File: C10con.kicad_sch (KiCad schematic)
At the start: 23 parts, among them IC1 TPS2553DRVT, J2 Conn_01x16_Male, J5 Conn_01x08_Male, U5 MIC5205-3.3YM5

Commit message: mod: part #
Parts:
- C17: Mouser 963-MAJCU168BB7104KT -> (none)
- C19, C20: Mouser 963-JMK316ABJ107ML-T -> (none)
- R28: Mouser 603-RC0603FR-073K3L -> (none)
- R9: Mouser 603-AC0603FR-07100KL -> (none)
Changed lines of the file:
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@@
 			)
 		)
-		(property "Description" "3.3kOhms, 1%, 1/10W"
-			(at 245.11 58.42 90)
-			(effects
-				(font
-					(size 1.27 1.27)
-				)
-				(hide yes)
-			)
-		)
-		(property "Mouser" "603-RC0603FR-073K3L"
+		(property "Description" "-55℃~+155℃ 100mW 3.3kΩ 75V Thick Film Resistor ±1% ±100ppm/℃ 0603 Chip Resistor - Surface Mount ROHS"
 			(at 245.11 58.42 90)
 			(effects
@@
 			)
 		)
-		(property "Description" "100kOhms, 1%, 1/10W"
-			(at 184.15 110.49 90)
-			(effects
-				(font
-					(size 1.27 1.27)
-				)
-				(hide yes)
-			)
-		)
-		(property "Mouser" "603-AC0603FR-07100KL"
+		(property "Description" "-55℃~+155℃ 100kΩ 100mW 75V Thick Film Resistor ±1% ±100ppm/℃ 0603 Chip Resistor - Surface Mount ROHS"
 			(at 184.15 110.49 90)
 			(effects
@@
 			)
 		)
-		(property "Description" "50V 0.1uF 0603 X7R"
-			(at 190.5 116.84 0)
-			(effects
-				(font
-					(size 1.27 1.27)
-				)
-				(hide yes)
-			)
-		)
-		(property "Mouser" "963-MAJCU168BB7104KT"
+		(property "Description" "100nF 50V X7R ±10% 0603 Multilayer Ceramic Capacitors MLCC - SMD/SMT ROHS100nF 50V X7R ±10% 0603 Multilayer Ceramic Capacitors MLCC - SMD/SMT ROHS"
 			(at 190.5 116.84 0)
 			(effects
@@
 		)
 		(property "Description" "6.3V 100uF X5R 1206 20%"
-			(at 232.41 116.84 0)
-			(effects
-				(font
-					(size 1.27 1.27)
-				)
-				(hide yes)
-			)
-		)
-		(property "Mouser" "963-JMK316ABJ107ML-T"
 			(at 232.41 116.84 0)
 			(effects
@@
 			(at 227.33 116.84 0)
 			(effects
-				(font
-					(size 1.27 1.27)
-				)
-				(hide yes)
-			)
-		)
-		(property "Mouser" "963-JMK316ABJ107ML-T"
-			(at 227.33 116.84 0)
-			(effects

Commit message: update: JLCPCB parts
Parts:
- IC1: LCSC Part # C2871420 -> C138719
- R10: value 18k -> 22k; LCSC Part # C25810 -> C31850
Other:
- note added: "R10=22k: ~1.1A limit"
- note removed: "R10=18k: ~1.4A limit"
