File: C10usb.kicad_sch (KiCad schematic)
At the start: 26 parts, among them J1 USB_B_Mini, U6 FT230XQ, U7 ISO7742

Commit message: mod: part #
Parts:
- R15: Mouser 71-CRCW0603-4.7K-E3 -> (none)
- R22, R23: Mouser 603-RC0603FR-073K3L -> (none)
Changed lines of the file:
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@@
 			)
 		)
-		(property "Description" "1/10watt 3.3Kohms 1%"
-			(at 162.56 83.82 90)
-			(effects
-				(font
-					(size 1.27 1.27)
-				)
-				(hide yes)
-			)
-		)
-		(property "Mouser" ""
+		(property "Description" "-55℃~+155℃ 100mW 3.3kΩ 75V Thick Film Resistor ±1% ±100ppm/℃ 0603 Chip Resistor - Surface Mount ROHS"
 			(at 162.56 83.82 90)
 			(effects
@@
 			)
 		)
-		(property "Description" "1/10watt 3.3Kohms 1%"
-			(at 162.56 74.93 90)
-			(effects
-				(font
-					(size 1.27 1.27)
-				)
-				(hide yes)
-			)
-		)
-		(property "Mouser" ""
+		(property "Description" "-55℃~+155℃ 100mW 3.3kΩ 75V Thick Film Resistor ±1% ±100ppm/℃ 0603 Chip Resistor - Surface Mount ROHS"
 			(at 162.56 74.93 90)
 			(effects
@@
 			)
 		)
-		(property "Description" "3.3kOhms, 1%, 1/10W"
-			(at 162.56 105.41 90)
-			(effects
-				(font
-					(size 1.27 1.27)
-				)
-				(hide yes)
-			)
-		)
-		(property "Mouser" "603-RC0603FR-073K3L"
+		(property "Description" "-55℃~+155℃ 100mW 3.3kΩ 75V Thick Film Resistor ±1% ±100ppm/℃ 0603 Chip Resistor - Surface Mount ROHS"
 			(at 162.56 105.41 90)
 			(effects
@@
 			)
 		)
-		(property "Description" "3.3kOhms, 1%, 1/10W"
-			(at 162.56 116.84 90)
-			(effects
-				(font
-					(size 1.27 1.27)
-				)
-				(hide yes)
-			)
-		)
-		(property "Mouser" "603-RC0603FR-073K3L"
+		(property "Description" "-55℃~+155℃ 100mW 3.3kΩ 75V Thick Film Resistor ±1% ±100ppm/℃ 0603 Chip Resistor - Surface Mount ROHS"
 			(at 162.56 116.84 90)
 			(effects
@@
 			)
 		)
-		(property "Description" "1/10watt 3.3Kohms 1%"
+		(property "Description" "-55℃~+155℃ 100mW 3.3kΩ 75V Thick Film Resistor ±1% ±100ppm/℃ 0603 Chip Resistor - Surface Mount ROHS"
 			(at 44.45 86.36 90)
 			(effects
-				(font
-					(size 1.27 1.27)
-				)
-				(hide yes)
-			)
-		)
-		(property "Mouser" "71-CRCW0603-4.7K-E3"
-			(at 44.45 86.36 90)
-			(effects
